Commit message: roda boba nos robôs e câmera para auxiliar na navegação dos robôs

File: vss_simulation/urdf/camera.urdf.xacro (robot description, xacro)
@@ -1,50 +1,64 @@
 <?xml version="1.0"?>
 <robot name="up_camera" xmlns:xacro="http://wiki.ros.org/xacro">
-    <link name="camera_base_link">
-        <visual>
-            <geometry>
-                <box size="0.05 0.05 0.05"/>
-            </geometry>
-            <material name="camera_material">
-                <color rgba="0 0.5 0.5 1"/>
-            </material>
-        </visual>
-    </link>
-    <link name="camera_link">
-        <visual>
-            <geometry>
-                <box size="0.02 0.02 0.02"/>
-            </geometry>
-            <material name="lens_material">
-                <color rgba="0 0 0 1"/>
-            </material>
-        </visual>
-    </link>
-    <joint name="camera_joint" type="fixed">
-        <parent link="camera_base_link"/>
-        <child link="camera_link"/>
-        <origin xyz="0 0 0" rpy="0 1.5708 0"/>
-    </joint>
-    <gazebo reference="camera_link">
-        <sensor name="camera" type="camera">
-            <pose>0 0 5 0 0 0</pose>
-            <visualize>true</visualize>
-            <update_rate>30</update_rate>
-            <camera>
-                <horizontal_fov>1.5708</horizontal_fov>
-                <image>
-                    <format>R8G8B8</format>
-                    <width>1920</width>
-                    <height>1080</height>
-                </image>
-                <clip>
-                    <near>1</near>
-                    <far>20</far>
-                </clip>
-            </camera>
-            <plugin name="camera_controller" filename="libgazebo_ros_camera.so">
-                <frame_name>camera_link</frame_name>
-            </plugin>
-        </sensor>
-    </gazebo>
+  <link name="camera_link">
+    <inertial>
+      <origin xyz="0 0 0" rpy="0 0 0"/>
+      <mass value="0.5"/>
+      <inertia ixx="0.001" ixy="0.0" ixz="0.0"
+               iyy="0.001" iyz="0.0"
+               izz="0.001"/>
+    </inertial>
+    <visual>
+      <origin xyz="0 0 0" rpy="0 0 0"/>
+      <geometry>
+        <box size="0.05 0.05 0.1"/>
+      </geometry>
+      <material name="black">
+        <color rgba="0 0.5 0.5 1"/>
+      </material>
+    </visual>
+    <collision>
+      <origin xyz="0 0 0" rpy="0 0 0"/>
+      <geometry>
+        <box size="0.05 0.05 0.1"/>
+      </geometry>
+    </collision>
+  </link>
+  <gazebo reference="camera_link">
+    <gravity>0</gravity>
+  </gazebo>
+  <gazebo reference="camera_link">
+    <sensor type="camera" name="camera_sensor">
+      <pose>0 0 0 0 0 0</pose>
+      <update_rate>30</update_rate>
+      <camera>
+        <horizontal_fov>0.7</horizontal_fov>
+        <image>
+          <width>480</width>
+          <height>640</height>
+          <format>R8G8B8</format>
+        </image>
+        <clip>
+          <near>0.05</near>
+          <far>100</far>
+        </clip>
+      </camera>
+      <always_on>true</always_on>
+      <visualize>true</visualize>
+    </sensor>
+    <plugin name="camera_controller" filename="libgazebo_ros_camera.so">
+      <always_on>true</always_on>
+      <update_rate>30.0</update_rate>
+      <camera_name>up_camera</camera_name>
+      <image_topic_name>image_raw</image_topic_name>
+      <camera_info_topic_name>camera_info</camera_info_topic_name>
+      <frame_name>camera_link</frame_name>
+      <hack_baseline>0.07</hack_baseline>
+      <distortion_k1>0.0</distortion_k1>
+      <distortion_k2>0.0</distortion_k2>
+      <distortion_k3>0.0</distortion_k3>
+      <distortion_t1>0.0</distortion_t1>
+      <distortion_t2>0.0</distortion_t2>
+    </plugin>
+  </gazebo>
 </robot>

File: vss_simulation/urdf/vss.urdf.xacro (robot description, xacro)
@@ -3,4 +3,5 @@
   <xacro:include filename="$(find vss_simulation)/urdf/common_properties.urdf.xacro" />
   <xacro:include filename="$(find vss_simulation)/urdf/inertias.urdf.xacro" />
+  <xacro:include filename="$(find vss_simulation)/urdf/roda_boba.urdf.xacro" />
   <xacro:macro name="vss_wheel_macro" params="base_size_x dir reflect mass width radius absolute_center_height">
   <link name="wheel${dir}_link">
@@ -80,4 +81,18 @@
       absolute_center_height="${wheel_radius}"
     />
+    <xacro:roda_boba_macro
+    prefix="front"
+    parent="base_link"
+    x_offset="0"
+    y_offset="${pos_y_roda_boba}"
+    z_offset="${pos_z_roda_boba}"
+    />
+    <xacro:roda_boba_macro
+    prefix="rear"
+    parent="base_link"
+    x_offset="0"
+    y_offset="${-pos_y_roda_boba}"
+    z_offset="${pos_z_roda_boba}"
+    />
   </xacro:macro>
 </robot>

File: vss_simulation/urdf/vss.xacro (robot description, xacro)
@@ -3,11 +3,16 @@
   <!-- 1) Definição dos parâmetros via property -->
   <xacro:property name="base_mass"    value="2.0"/>
-  <xacro:property name="base_size_x"  value="0.055"/> <!-- rodas tem eixo paralelo ao X -->
+  <xacro:property name="base_size_x"  value="0.055"/> <!-- rodas estão paralelas ao eixo X -->
   <xacro:property name="base_size_y"  value="0.075"/>
-  <xacro:property name="base_size_z"  value="0.065"/> <!-- a vertical é o eixo Y -->
+  <xacro:property name="base_size_z"  value="0.065"/> <!-- a vertical é o eixo Z -->
   <xacro:property name="wheel_mass"  value="0.1"/>
   <xacro:property name="wheel_width"  value="0.01"/>
   <xacro:property name="wheel_radius" value="0.02"/>
   <xacro:property name="wheel_center_height"  value="0.01"/>  <!-- value="0" é a parte de baixo da base -->
+  <!-- Roda boba-->
+  <xacro:property name="raio_roda_boba" value="0.01" />
+  <xacro:property name="massa_roda_boba" value="0.05" />
+  <xacro:property name="pos_y_roda_boba" value="${base_size_y/2 - raio_roda_boba - 0.005}" />
+  <xacro:property name="pos_z_roda_boba" value="${raio_roda_boba}" />
   <!-- 3) Inclui definição da sua macro de montagem -->
   <xacro:include filename="$(find vss_simulation)/urdf/vss.urdf.xacro"/>
