Commit message: Adicionei as rodas ao robo

File: vss_simulation/urdf/vss.urdf.xacro (robot description, xacro)
@@ -3,5 +3,33 @@
   <xacro:include filename="$(find vss_simulation)/urdf/common_properties.urdf.xacro" />
   <xacro:include filename="$(find vss_simulation)/urdf/inertias.urdf.xacro" />
-  <xacro:macro name="vss_base_macro" params="mass size_x size_y size_z">
+  <xacro:macro name="vss_wheel_macro" params="base_size_x dir reflect mass width radius absolute_center_height">
+  <link name="wheel${dir}_link">
+      <visual>
+        <origin xyz="${reflect*width/2} 0 0" rpy="0 1.57 0"/>
+        <geometry>
+          <cylinder radius="${radius}" length="${width}"/>
+        </geometry>
+      </visual>
+      <collision>
+        <origin xyz="${reflect*width/2} 0 0" rpy="0 1.57 0"/>
+        <geometry>
+          <cylinder radius="${radius}" length="${width}"/>
+        </geometry>
+      </collision>
+      <xacro:cylinder_inertia_macro mass="${mass}" radius="${radius}" length="${width}"/>
+      <gazebo>
+        <material>Gazebo/Blue</material>
+        <mu1>0.2</mu1>
+        <mu2>0.2</mu2>
+      </gazebo>
+    </link>
+     <joint name="base_to_wheel${dir}" type="continuous">
+        <parent link="base_link"/>
+        <child link="wheel${dir}_link"/>
+        <axis xyz="1 0 0"/>
+        <origin xyz="${reflect*(base_size_x/2)} 0 ${absolute_center_height}" />
+    </joint>
+  </xacro:macro>
+  <xacro:macro name="vss_base_macro" params="mass size_x size_y size_z wheel_mass wheel_width wheel_radius wheel_center_height">
     <link name="base_link">
       <visual>
@@ -24,4 +52,22 @@
       </gazebo>
     </link>
+    <xacro:vss_wheel_macro
+      base_size_x="${base_size_x}"
+      dir = "R"
+      reflect = "1"
+      mass="${wheel_mass}"
+      width="${wheel_width}"
+      radius="${wheel_radius}"
+      absolute_center_height="${wheel_center_height-(base_size_y/2)}"
+    />
+    <xacro:vss_wheel_macro
+      base_size_x="${base_size_x}"
+      dir = "L"
+      reflect = "-1"
+      mass="${wheel_mass}"
+      width="${wheel_width}"
+      radius="${wheel_radius}"
+      absolute_center_height="${wheel_center_height-(base_size_y/2)}"
+    />
   </xacro:macro>
 </robot>

File: vss_simulation/urdf/vss.xacro (robot description, xacro)
@@ -6,4 +6,8 @@
   <xacro:property name="base_size_y"  value="0.075"/>
   <xacro:property name="base_size_z"  value="0.075"/>
+  <xacro:property name="wheel_mass"  value="0.1"/>
+  <xacro:property name="wheel_width"  value="0.01"/>
+  <xacro:property name="wheel_radius" value="0.02"/>
+  <xacro:property name="wheel_center_height"  value="0.01"/>  <!-- value="0" é a parte de baixo da base -->
   <!-- 3) Inclui definição da sua macro de montagem -->
   <xacro:include filename="$(find vss_simulation)/urdf/vss.urdf.xacro"/>
@@ -14,4 +18,8 @@
     size_y="${base_size_y}"
     size_z="${base_size_z}"
+    wheel_mass="${wheel_mass}"
+    wheel_width="${wheel_width}"
+    wheel_radius="${wheel_radius}"
+    wheel_center_height="${wheel_center_height}"
   />
 </robot>

Commit message: Adicionei os materiais no vss

File: vss_simulation/urdf/vss.urdf.xacro (robot description, xacro)
@@ -10,4 +10,5 @@
           <cylinder radius="${radius}" length="${width}"/>
         </geometry>
+        <material name="black"/>
       </visual>
       <collision>
@@ -19,5 +20,5 @@
       <xacro:cylinder_inertia_macro mass="${mass}" radius="${radius}" length="${width}"/>
       <gazebo>
-        <material>Gazebo/Blue</material>
+        <material>Gazebo/Black</material>
         <mu1>0.2</mu1>
         <mu2>0.2</mu2>
@@ -38,4 +39,5 @@
           <box size="${size_x} ${size_y} ${size_z}"/>
         </geometry>
+        <material name="blue"/>
       </visual>
       <collision>

Commit message: Corrigi a altura do vss

File: vss_simulation/urdf/vss.urdf.xacro (robot description, xacro)
@@ -35,7 +35,7 @@
     <link name="base_link">
       <visual>
-        <origin xyz="0 0 0" rpy="0 0 0"/>
+        <origin xyz="0 0 ${wheel_radius-wheel_center_height+size_z/2}" rpy="0 0 0"/>
         <geometry>
-          <box size="${size_x} ${size_y} ${size_z}"/>
+          <box size="${size_y} ${size_x} ${size_z}"/>
         </geometry>
         <material name="blue"/>
@@ -44,5 +44,5 @@
         <origin xyz="0 0 0" rpy="0 0 0"/>
         <geometry>
-          <box size="${size_x} ${size_y} ${size_z}"/>
+          <box size="${size_y} ${size_x} ${size_z}"/>
         </geometry>
       </collision>
@@ -61,5 +61,5 @@
       width="${wheel_width}"
       radius="${wheel_radius}"
-      absolute_center_height="${wheel_center_height-(base_size_y/2)}"
+      absolute_center_height="${wheel_radius}"
     />
     <xacro:vss_wheel_macro
@@ -70,5 +70,5 @@
       width="${wheel_width}"
       radius="${wheel_radius}"
-      absolute_center_height="${wheel_center_height-(base_size_y/2)}"
+      absolute_center_height="${wheel_radius}"
     />
   </xacro:macro>

Commit message: Corrigi as dimensões do robo e o sentido de rotacao das rodas

File: vss_simulation/urdf/vss.urdf.xacro (robot description, xacro)
@@ -28,5 +28,5 @@
         <parent link="base_link"/>
         <child link="wheel${dir}_link"/>
-        <axis xyz="1 0 0"/>
+        <axis xyz="-1 0 0"/>
         <origin xyz="${reflect*(base_size_x/2)} 0 ${absolute_center_height}" />
     </joint>
@@ -37,5 +37,5 @@
         <origin xyz="0 0 ${wheel_radius-wheel_center_height+size_z/2}" rpy="0 0 0"/>
         <geometry>
-          <box size="${size_y} ${size_x} ${size_z}"/>
+          <box size="${size_x} ${size_y} ${size_z}"/>
         </geometry>
         <material name="blue"/>
@@ -44,5 +44,5 @@
         <origin xyz="0 0 0" rpy="0 0 0"/>
         <geometry>
-          <box size="${size_y} ${size_x} ${size_z}"/>
+          <box size="${size_x} ${size_y} ${size_z}"/>
         </geometry>
       </collision>

File: vss_simulation/urdf/vss.xacro (robot description, xacro)
@@ -3,7 +3,7 @@
   <!-- 1) Definição dos parâmetros via property -->
   <xacro:property name="base_mass"    value="2.0"/>
-  <xacro:property name="base_size_x"  value="0.075"/>
+  <xacro:property name="base_size_x"  value="0.055"/> <!-- rodas tem eixo paralelo ao X -->
   <xacro:property name="base_size_y"  value="0.075"/>
-  <xacro:property name="base_size_z"  value="0.075"/>
+  <xacro:property name="base_size_z"  value="0.065"/> <!-- a vertical é o eixo Y -->
   <xacro:property name="wheel_mass"  value="0.1"/>
   <xacro:property name="wheel_width"  value="0.01"/>

Commit message: consertei a inercia e adicionei launch do robos

File: vss_simulation/urdf/vss.urdf.xacro (robot description, xacro)
@@ -18,5 +18,9 @@
         </geometry>
       </collision>
-      <xacro:cylinder_inertia_macro mass="${mass}" radius="${radius}" length="${width}"/>
+      <inertial>
+        <origin xyz="${reflect*width/2} 0 0" rpy="0 1.57 0"/>
+        <mass value="${mass}"/>
+        <xacro:cylinder_inertia_macro mass="${mass}" radius="${radius}" length="${width}"/>
+      </inertial>
       <gazebo>
         <material>Gazebo/Black</material>
@@ -42,10 +46,14 @@
       </visual>
       <collision>
-        <origin xyz="0 0 0" rpy="0 0 0"/>
+        <origin xyz="0 0 ${wheel_radius-wheel_center_height+size_z/2}" rpy="0 0 0"/>
         <geometry>
           <box size="${size_x} ${size_y} ${size_z}"/>
         </geometry>
       </collision>
-      <xacro:cuboid_inertia_macro mass="${mass}" width="${size_y}" length="${size_x}" height="${size_z}"/>
+      <inertial>
+        <origin xyz="0 0 ${wheel_radius-wheel_center_height+size_z/2}" rpy="0 0 0"/>
+        <mass value="${mass}"/>
+        <xacro:cuboid_inertia_macro mass="${mass}" width="${size_y}" length="${size_x}" height="${size_z}"/>
+      </inertial>
       <gazebo>
         <material>Gazebo/Blue</material>
@@ -55,5 +63,5 @@
     </link>
     <xacro:vss_wheel_macro
-      base_size_x="${base_size_x}"
+      base_size_x="${size_x}"
       dir = "R"
       reflect = "1"
@@ -64,5 +72,5 @@
     />
     <xacro:vss_wheel_macro
-      base_size_x="${base_size_x}"
+      base_size_x="${size_x}"
       dir = "L"
       reflect = "-1"

Commit message: usei argumento para passar o prefixo para o nome do robo, movi o macro da roda para outro arquivo

File: vss_simulation/urdf/vss.urdf.xacro (robot description, xacro)
@@ -4,39 +4,7 @@
   <xacro:include filename="$(find vss_simulation)/urdf/inertias.urdf.xacro" />
   <xacro:include filename="$(find vss_simulation)/urdf/roda_boba.urdf.xacro" />
-  <xacro:macro name="vss_wheel_macro" params="base_size_x dir reflect mass width radius absolute_center_height">
-  <link name="wheel${dir}_link">
-      <visual>
-        <origin xyz="${reflect*width/2} 0 0" rpy="0 1.57 0"/>
-        <geometry>
-          <cylinder radius="${radius}" length="${width}"/>
-        </geometry>
-        <material name="black"/>
-      </visual>
-      <collision>
-        <origin xyz="${reflect*width/2} 0 0" rpy="0 1.57 0"/>
-        <geometry>
-          <cylinder radius="${radius}" length="${width}"/>
-        </geometry>
-      </collision>
-      <inertial>
-        <origin xyz="${reflect*width/2} 0 0" rpy="0 1.57 0"/>
-        <mass value="${mass}"/>
-        <xacro:cylinder_inertia_macro mass="${mass}" radius="${radius}" length="${width}"/>
-      </inertial>
-      <gazebo>
-        <material>Gazebo/Black</material>
-        <mu1>0.2</mu1>
-        <mu2>0.2</mu2>
-      </gazebo>
-    </link>
-     <joint name="base_to_wheel${dir}" type="continuous">
-        <parent link="base_link"/>
-        <child link="wheel${dir}_link"/>
-        <axis xyz="-1 0 0"/>
-        <origin xyz="${reflect*(base_size_x/2)} 0 ${absolute_center_height}" />
-    </joint>
-  </xacro:macro>
-  <xacro:macro name="vss_base_macro" params="mass size_x size_y size_z wheel_mass wheel_width wheel_radius wheel_center_height">
-    <link name="base_link">
+  <xacro:include filename="$(find vss_simulation)/urdf/wheel.urdf.xacro"/>
+  <xacro:macro name="vss_base_macro" params="prefix mass size_x size_y size_z wheel_mass wheel_width wheel_radius wheel_center_height">
+    <link name="${prefix}base_link">
       <visual>
         <origin xyz="0 0 ${wheel_radius-wheel_center_height+size_z/2}" rpy="0 0 0"/>
@@ -64,6 +32,7 @@
     </link>
     <xacro:vss_wheel_macro
+      prefix="${prefix}R_"
+      parent="${prefix}base_link"
       base_size_x="${base_size_x}"
-      dir = "R"
       reflect = "1"
       mass="${wheel_mass}"
@@ -73,6 +42,7 @@
     />
     <xacro:vss_wheel_macro
+      prefix="${prefix}L_"
+      parent="${prefix}base_link"
       base_size_x="${base_size_x}"
-      dir = "L"
       reflect = "-1"
       mass="${wheel_mass}"
@@ -82,6 +52,6 @@
     />
     <xacro:roda_boba_macro
-    prefix="front"
-    parent="base_link"
+    prefix="${prefix}front_"
+    parent="${prefix}base_link"
     x_offset="0"
     y_offset="${pos_y_roda_boba}"
@@ -89,6 +59,6 @@
     />
     <xacro:roda_boba_macro
-    prefix="rear"
-    parent="base_link"
+    prefix="${prefix}rear_"
+    parent="${prefix}base_link"
     x_offset="0"
     y_offset="${-pos_y_roda_boba}"

File: vss_simulation/urdf/vss.xacro (robot description, xacro)
@@ -1,4 +1,6 @@
 <?xml version="1.0"?>
 <robot name="vss_robot_model" xmlns:xacro="http://www.ros.org/wiki/xacro">
+  <!-- 0) Obtençao de parâmetros especificos via args-->
+  <xacro:arg name="prefix" default="vss_"/>
   <!-- 1) Definição dos parâmetros via property -->
   <xacro:property name="base_mass"    value="2.0"/>
@@ -19,4 +21,5 @@
   <!-- 4) Invoca a macro com os valores acima -->
   <xacro:vss_base_macro
+    prefix="$(arg prefix)"
     mass="${base_mass}"
     size_x="${base_size_x}"
